Commit message: Add multi-joint trajectory client with CSV support
- Multi-joint trajectory client for 3-joint robotic system
- Action server name configurable via parameter
- CSV-based velocity profile support
- Reads initial joint positions from /joint_states
- Updated system to support waist, shoulder, and elbow joints
- Renamed controller to kinematic_controller_baseline
- Added deliverables folder for easy integration

File: urdf/stepper.urdf.xacro (robot description, xacro)
@@ -16,6 +16,6 @@
     </visual>
   </link>
-  <!-- Stepper motor link -->
-  <link name="stepper_link">
+  <!-- Waist link (was stepper_link) -->
+  <link name="waist_link">
     <visual>
       <geometry>
@@ -27,8 +27,44 @@
     </visual>
   </link>
-  <!-- Joint connecting base to stepper -->
-  <joint name="stepper_joint" type="continuous">
+  <!-- Waist joint (was stepper_joint) -->
+  <joint name="waist_joint" type="continuous">
     <parent link="base_link"/>
-    <child link="stepper_link"/>
+    <child link="waist_link"/>
+    <origin xyz="0 0 0.05" rpy="0 0 0"/>
+    <axis xyz="0 0 1"/>
+  </joint>
+  <!-- Shoulder link -->
+  <link name="shoulder_link">
+    <visual>
+      <geometry>
+        <cylinder length="0.05" radius="0.03"/>
+      </geometry>
+      <material name="red">
+        <color rgba="0.8 0 0 1"/>
+      </material>
+    </visual>
+  </link>
+  <!-- Shoulder joint -->
+  <joint name="shoulder_joint" type="continuous">
+    <parent link="waist_link"/>
+    <child link="shoulder_link"/>
+    <origin xyz="0 0 0.05" rpy="0 0 0"/>
+    <axis xyz="0 0 1"/>
+  </joint>
+  <!-- Elbow link -->
+  <link name="elbow_link">
+    <visual>
+      <geometry>
+        <cylinder length="0.05" radius="0.03"/>
+      </geometry>
+      <material name="green">
+        <color rgba="0 0.8 0 1"/>
+      </material>
+    </visual>
+  </link>
+  <!-- Elbow joint -->
+  <joint name="elbow_joint" type="continuous">
+    <parent link="shoulder_link"/>
+    <child link="elbow_link"/>
     <origin xyz="0 0 0.05" rpy="0 0 0"/>
     <axis xyz="0 0 1"/>
@@ -43,5 +79,21 @@
       <param name="microsteps">$(arg microsteps)</param>
     </hardware>
-    <joint name="stepper_joint">
+    <joint name="waist_joint">
+      <command_interface name="velocity">
+        <param name="min">-50</param>
+        <param name="max">50</param>
+      </command_interface>
+      <state_interface name="position"/>
+      <state_interface name="velocity"/>
+    </joint>
+    <joint name="shoulder_joint">
+      <command_interface name="velocity">
+        <param name="min">-50</param>
+        <param name="max">50</param>
+      </command_interface>
+      <state_interface name="position"/>
+      <state_interface name="velocity"/>
+    </joint>
+    <joint name="elbow_joint">
       <command_interface name="velocity">
         <param name="min">-50</param>
